File: midimania.kicad_sch (KiCad schematic)
At the start: 21 parts, among them J1 Conn_01x01_Female, J10 Conn_01x01_Female, J11 Conn_01x01_Female, J12 Conn_01x01_Female, J2 Conn_01x01_Female, J3 Conn_01x01_Female, J4 Conn_01x01_Female, J5 Conn_01x01_Female, J6 Conn_01x01_Female, J7 Conn_01x01_Female, J8 Conn_01x01_Female, J9 Conn_01x01_Female, U1 Teensy3.2

Commit message: pcb design
Connections:
- net l1: now also U1.21 (14_A0_SCK); no longer U1.28 (21_A7_RX1_CS_PWM)
- net l2: now also U1.22 (15_A1_CS_Touch); no longer U1.27 (20_A6_CS_PWM)
- net l3: now also U1.23 (16_A2_SCL0_Touch); no longer U1.26 (19_A5_SCL0_Touch)
- net l4: now also U1.24 (17_A3_SDA0_Touch); no longer U1.25 (18_A4_SDA0_Touch)
- net p1: now also U1.28 (21_A7_RX1_CS_PWM); no longer U1.21 (14_A0_SCK)
- net p2: now also U1.27 (20_A6_CS_PWM); no longer U1.22 (15_A1_CS_Touch)
- net p3: now also U1.26 (19_A5_SCL0_Touch); no longer U1.23 (16_A2_SCL0_Touch)
- net p4: now also U1.25 (18_A4_SDA0_Touch); no longer U1.24 (17_A3_SDA0_Touch)
Changed lines of the file:
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@@
     (effects (font (size 1.27 1.27)) (justify left bottom))
   )
-  (label "p2" (at 26.67 82.55 0)
+  (label "l2" (at 26.67 82.55 0)
     (effects (font (size 1.27 1.27)) (justify left bottom))
   )
-  (label "l2" (at 26.67 95.25 0)
+  (label "p2" (at 26.67 95.25 0)
     (effects (font (size 1.27 1.27)) (justify left bottom))
   )
@@
     (effects (font (size 1.27 1.27)) (justify left bottom))
   )
-  (label "p1" (at 26.67 80.01 0)
+  (label "l1" (at 26.67 80.01 0)
     (effects (font (size 1.27 1.27)) (justify left bottom))
   )
-  (label "p3" (at 26.67 85.09 0)
+  (label "l3" (at 26.67 85.09 0)
     (effects (font (size 1.27 1.27)) (justify left bottom))
   )
@@
     (effects (font (size 1.27 1.27)) (justify left bottom))
   )
-  (label "l1" (at 26.67 97.79 0)
+  (label "p1" (at 26.67 97.79 0)
     (effects (font (size 1.27 1.27)) (justify left bottom))
   )
@@
     (effects (font (size 1.27 1.27)) (justify left bottom))
   )
-  (label "l3" (at 26.67 92.71 0)
+  (label "p3" (at 26.67 92.71 0)
     (effects (font (size 1.27 1.27)) (justify left bottom))
   )
@@
     (effects (font (size 1.27 1.27)) (justify left bottom))
   )
-  (label "p4" (at 26.67 87.63 0)
+  (label "l4" (at 26.67 87.63 0)
     (effects (font (size 1.27 1.27)) (justify left bottom))
   )
-  (label "l4" (at 26.67 90.17 0)
+  (label "p4" (at 26.67 90.17 0)
     (effects (font (size 1.27 1.27)) (justify left bottom))
   )
